File: ece312-final-project.kicad_sch (KiCad schematic)
At the start: 4 parts, among them U1 ATmega328-P, Y1 32.768KHz Crystal

Commit message: Finalized Schematic
Parts:
- removed Y1: 32.768KHz Crystal, symbol Device:Crystal
Connections:
- net Gesture Sensor/G1 is gone; now on net Gesture Sensor/G0: U1.26 (PC3)
- net Gesture Sensor/G0: no longer U1.25 (PC2)
- net LCD/D4: now also U1.2 (PD0); no longer U1.5 (PD3)
- net LCD/D5: now also U1.3 (PD1); no longer U1.4 (PD2)
- net LCD/D6: now also U1.4 (PD2); no longer U1.3 (PD1)
- net LCD/D7: now also U1.5 (PD3); no longer U1.2 (PD0)
- net Audio System/PWM/SHDWN: no longer names the net of U1.12 (PD6)
- net Audio System/SCL: no longer names the net of U1.28 (PC5)
- net Audio System/SDA: no longer names the net of U1.27 (PC4)
- net GNDREF renamed GND
Other:
- sheet Audio System ports: added none; removed PWM/SHDWN, SCL, SDA
- sheet Gesture Sensor ports: added none; removed G1
- moved on the sheet: D1, R1, U1

Commit message: Added audio sheet pins
Connections:
- net Audio System/PWM/SEL0: now reaches U1.12 (PD6)
- net Audio System/PLAYPAUSE: now reaches U1.27 (PC4)
- net Audio System/SEL1: now reaches U1.28 (PC5)
Other:
- sheet Audio System ports: added PLAYPAUSE, PWM/SEL0, SEL1; removed none
Changed lines of the file:
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@@
+      (effects (font (size 1.27 1.27)) (justify right))
+    )
+    (pin "PLAYPAUSE" input (at 124.46 121.92 90)
+      (effects (font (size 1.27 1.27)) (justify right))
+    )
+    (pin "PWM{slash}SEL0" input (at 119.38 121.92 90)
+      (effects (font (size 1.27 1.27)) (justify right))
+    )
+    (pin "SEL1" input (at 121.92 121.92 90)
       (effects (font (size 1.27 1.27)) (justify right))
     )
