File: audio_system.kicad_sch (KiCad schematic)
At the start: 8 parts, among them U2 MCP4725xxx-xCH, U3 MAX98306xDT

Commit message: Finalized Schematic
Parts:
- removed R8: 10k, symbol Device:R
- removed U2: MCP4725xxx-xCH, Package_TO_SOT_SMD:SOT-23-6, symbol Analog_DAC:MCP4725xxx-xCH
- added U5: NUCLEO-32L432KC, Package_DFN_QFN:QFN-32-1EP_5x5mm_P0.5mm_EP3.45x3.45mm, symbol MCU_ST_STM32L4:STM32L432KBUx
- U3: value MAX98306xDT -> Adafruit-MAX98306
Connections:
- net +5V: now also U5.1 (VDD), U5.16 (VSS), U5.17 (VDD), U5.32 (VSS), U5.33 (VSS)
- net at U3.3 (INL+), U3.7 (INR+): now also U5.10 (PA4)
- net PWM/SHDWN renamed PLAYPAUSE
- net PLAYPAUSE: no longer BZ1.1 (-)
- net SCL renamed PWM/SEL0
- net PWM/SEL0: now also BZ1.1 (-), U5.28 (PB5)
- net SDA renamed SEL1
- net SEL1: now also U5.27 (PB4)
Other:
- moved on the sheet: BZ1, R6, R7

Commit message: added pot for audio volume
Parts:
- added RV1: 10k, symbol Device:R_Potentiometer_US
Connections:
- net +5V: now also RV1.3
- net at U3.3 (INL+), U3.7 (INR+): now also RV1.1; no longer U5.10 (PA4)
- new net: RV1.2, U5.10 (PA4)
Changed lines of the file:
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@@
 (kicad_sch (version 20230121) (generator eeschema)
   (paper "A4")
+  (junction (at 102.87 49.53) (diameter 0) (color 0 0 0 0)
+  )
   (junction (at 105.41 57.15) (diameter 0) (color 0 0 0 0)
   )
@@
   )
   (junction (at 41.91 59.69) (diameter 0) (color 0 0 0 0)
-  )
-  (junction (at 102.87 49.53) (diameter 0) (color 0 0 0 0)
   )
   (no_connect (at 33.02 99.06))
@@
     (stroke (width 0) (type default))
   )
+  (wire (pts (xy 73.66 44.45) (xy 99.06 44.45))
+    (stroke (width 0) (type default))
+  )
   (wire (pts (xy 105.41 52.07) (xy 105.41 57.15))
     (stroke (width 0) (type default))
@@
     (stroke (width 0) (type default))
   )
+  (wire (pts (xy 96.52 33.02) (xy 96.52 36.83))
+    (stroke (width 0) (type default))
+  )
   (wire (pts (xy 123.19 73.66) (xy 123.19 69.85))
     (stroke (width 0) (type default))
@@
     (stroke (width 0) (type default))
   )
-  (wire (pts (xy 102.87 44.45) (xy 102.87 49.53))
+  (wire (pts (xy 102.87 40.64) (xy 102.87 33.02))
     (stroke (width 0) (type default))
   )
@@
     (stroke (width 0) (type default))
   )
-  (wire (pts (xy 73.66 44.45) (xy 102.87 44.45))
-    (stroke (width 0) (type default))
-  )
   (wire (pts (xy 110.49 52.07) (xy 105.41 52.07))
     (stroke (width 0) (type default))
   )
   (wire (pts (xy 102.87 49.53) (xy 102.87 54.61))
+    (stroke (width 0) (type default))
+  )
+  (wire (pts (xy 102.87 33.02) (xy 96.52 33.02))
+    (stroke (width 0) (type default))
+  )
+  (wire (pts (xy 102.87 48.26) (xy 102.87 49.53))
     (stroke (width 0) (type default))
   )
@@
   (hierarchical_label "PWM{slash}SEL0" (shape input) (at 29.21 62.23 180) (fields_autoplaced)
     (effects (font (size 1.27 1.27)) (justify right))
+  )
+  (symbol (lib_id "power:GND") (at 96.52 36.83 0) (unit 1)
+    (in_bom yes) (on_board yes) (dnp no)
+    (property "Reference" "#PWR023" (at 96.52 43.18 0)
+      (effects (font (size 1.27 1.27)) hide)
+    )
+    (property "Value" "GND" (at 96.52 40.64 0)
+      (effects (font (size 1.27 1.27)))
+    )
+    (property "Footprint" "" (at 96.52 36.83 0)
+      (effects (font (size 1.27 1.27)) hide)
+    )
+    (property "Datasheet" "" (at 96.52 36.83 0)
+      (effects (font (size 1.27 1.27)) hide)
+    )
+    (pin "1")
+    (instances
+      (project "ece312-final-project"
+        (path "/fafbac94-05bd-4749-8502-4886ccc0ec35/141be4a4-2435-4801-9a0f-ad0c10bfe2e5"
+          (reference "#PWR023") (unit 1)
+        )
+      )
+    )
   )
   (symbol (lib_id "power:+5V") (at 76.2 97.79 0) (unit 1)
@@
         )
       )
+    )
+  )
+  (symbol (lib_id "Device:R_Potentiometer_US") (at 102.87 44.45 180) (unit 1)
+    (in_bom yes) (on_board yes) (dnp no)
+    (property "Reference" "RV1" (at 105.41 45.7201 90)
+      (effects (font (size 1.27 1.27)) (justify right))
+    )
+    (property "Value" "10k" (at 107.95 45.72 90)
+      (effects (font (size 1.27 1.27)) (justify right))
+    )
+    (property "Footprint" "" (at 102.87 44.45 0)
+      (effects (font (size 1.27 1.27)) hide)
+    )
+    (property "Datasheet" "~" (at 102.87 44.45 0)
+      (effects (font (size 1.27 1.27)) hide)
+    )
+    (pin "1")
+    (pin "2")
+    (pin "3")
+    (instances
+      (project "ece312-final-project"
+        (path "/fafbac94-05bd-4749-8502-4886ccc0ec35/2a0acbe2-314c-45ae-b756-7238c9fcb4d8"
+          (reference "RV1") (unit 1)
+        )
+        (path "/fafbac94-05bd-4749-8502-4886ccc0ec35/141be4a4-2435-4801-9a0f-ad0c10bfe2e5"
+          (reference "RV2") (unit 1)
+        )
+      )
